Commit message: Resolve merge conflicts: Keep full RoboDK integration features

File: assets/design_export.urdf (robot description, URDF)
Before this commit: robot robot, 1 links, 0 joints
Links:
- removed link base_link
- added link ABB CRB 1300-7/1.4, mass 1; collision box size=0.1 0.1 0.1; visual box size=0.1 0.1 0.1
